File: hardware/funbox_v3_midi_exp/Power.kicad_sch (KiCad schematic)
At the start: 10 parts, among them U1 TL074, U2 L7805

Commit message: Updated schematic with new quad op amp
Parts:
- U1: value TL074 -> MCP6024
Changed lines of the file:
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@@
       (effects (font (size 1.27 1.27)) (justify left))
     )
-    (property "Value" "TL074" (at 176.53 105.41 0)
+    (property "Value" "MCP6024" (at 176.53 105.41 0)
       (effects (font (size 1.27 1.27)) (justify left))
     )
